File: PolluxWakeupShield/PolluxWakeupShield.brd (EAGLE design)
At the start: 73.7 x 53.3 mm, 16 parts, among them U1 ARDUINO_SHIELD

Commit message: dd last schematics with xbee improvement
Parts:
- moved ALIM 10.2 mm to (44.5, 21.6)
- moved U$2 1.27 mm to (37.5, 21.6)
Connections:
- net N$2: now also U1.D9; no longer U1.D7
- net N$3: now also U1.D10; no longer U1.D8
- net N$4: now also U1.D11; no longer U1.D9
Routing:
- net WAKEUP: track 94.6 -> 77.0 mm
- net GND: track 17.4 -> 30.1 mm
- net 5V: track 109.1 -> 118.0 mm
- net N$2: track 32.9 -> 27.3 mm
- net N$3: track 38.7 -> 34.4 mm
- net N$4: track 45.1 -> 40.7 mm
- net SCL: track 97.4 -> 99.5 mm
- net TX: track 96.2 -> 95.0 mm
- net SLEEP: track 67.0 -> 65.7 mm
- net RX: track 104.4 -> 103.1 mm
- net 3.3V: track 42.6 -> 41.3 mm
- net RESET: track 72.9 -> 71.7 mm
