File: PolluxWakeupShield/PolluxWakeupShield.sch (EAGLE design)
At the start: 16 parts, among them U1 ARDUINO_SHIELD

Commit message: dd last schematics with xbee improvement
Connections:
- net N$2: now also U1.*D9; no longer U1.D7
- net N$3: now also U1.*D10; no longer U1.D8
- net N$4: now also U1.*D11; no longer U1.*D9
Changed lines of the file:
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@@
 <net name="N$2" class="0">
 <segment>
-<pinref part="U1" gate="G$1" pin="D7"/>
-<wire x1="185.42" y1="137.16" x2="203.2" y2="137.16" width="0.1524" layer="91"/>
-<wire x1="203.2" y1="137.16" x2="203.2" y2="139.7" width="0.1524" layer="91"/>
 <pinref part="LED3" gate="G$1" pin="1"/>
 <wire x1="203.2" y1="139.7" x2="213.36" y2="139.7" width="0.1524" layer="91"/>
+<pinref part="U1" gate="G$1" pin="*D9"/>
+<wire x1="185.42" y1="132.08" x2="203.2" y2="132.08" width="0.1524" layer="91"/>
+<wire x1="203.2" y1="132.08" x2="203.2" y2="139.7" width="0.1524" layer="91"/>
 </segment>
 </net>
@@
 <segment>
 <pinref part="LED2" gate="G$1" pin="1"/>
-<wire x1="213.36" y1="132.08" x2="203.2" y2="132.08" width="0.1524" layer="91"/>
-<wire x1="203.2" y1="132.08" x2="203.2" y2="134.62" width="0.1524" layer="91"/>
-<pinref part="U1" gate="G$1" pin="D8"/>
-<wire x1="203.2" y1="134.62" x2="185.42" y2="134.62" width="0.1524" layer="91"/>
+<wire x1="213.36" y1="132.08" x2="205.74" y2="132.08" width="0.1524" layer="91"/>
+<pinref part="U1" gate="G$1" pin="*D10"/>
+<wire x1="185.42" y1="129.54" x2="205.74" y2="129.54" width="0.1524" layer="91"/>
+<wire x1="205.74" y1="129.54" x2="205.74" y2="132.08" width="0.1524" layer="91"/>
 </segment>
 </net>
 <net name="N$4" class="0">
 <segment>
-<pinref part="U1" gate="G$1" pin="*D9"/>
-<wire x1="185.42" y1="132.08" x2="200.66" y2="132.08" width="0.1524" layer="91"/>
-<wire x1="200.66" y1="132.08" x2="200.66" y2="124.46" width="0.1524" layer="91"/>
 <pinref part="LED1" gate="G$1" pin="1"/>
-<wire x1="200.66" y1="124.46" x2="213.36" y2="124.46" width="0.1524" layer="91"/>
+<wire x1="193.04" y1="124.46" x2="213.36" y2="124.46" width="0.1524" layer="91"/>
+<pinref part="U1" gate="G$1" pin="*D11"/>
+<wire x1="185.42" y1="127" x2="193.04" y2="127" width="0.1524" layer="91"/>
+<wire x1="193.04" y1="127" x2="193.04" y2="124.46" width="0.1524" layer="91"/>
 </segment>
 </net>
